Commit message: add the control of four wheel

File: car_model/robots/car_model.xacro (robot description, xacro)
@@ -138,5 +138,5 @@
     <origin rpy="0 1.57075 1.57075" xyz="${-car_a/2+0.02} ${-car_b/2-0.01} 0" />
     <limit effort="100" velocity="100" />
-    <joint_properties damping="0" friction="0.0" />
+    <joint_properties damping="0" friction="1.0" />
   </joint>
   <!-- #################### -->
@@ -179,5 +179,5 @@
     <origin rpy="0 1.57075 1.57075" xyz="${car_a/2-0.02} ${car_b/2+0.01} 0" />
     <limit effort="100" velocity="100" />
-    <joint_properties damping="0" friction="0.0" />
+    <joint_properties damping="0" friction="1.0" />
   </joint>
   <!-- #################### -->
@@ -220,5 +220,5 @@
     <origin rpy="0 1.57075 1.57075" xyz="${-car_a/2+0.02} ${car_b/2+0.01} 0" />
     <limit effort="100" velocity="100" />
-    <joint_properties damping="0" friction="0.0" />
+    <joint_properties damping="0" friction="1.0" />
   </joint>
   <!-- #################### -->
@@ -263,5 +263,5 @@
     <origin xyz="${car_a/2-column_width} 0 ${car_c}" />
     <limit effort="100" velocity="100" />
-    <joint_properties damping="0" friction="0.0" />
+    <joint_properties damping="0" friction="1.0" />
   </joint>
   <!-- #################### -->
@@ -454,4 +454,48 @@
     </joint>
     <actuator name="motor_column_link3">
+      <hardwareInterface>hardware_interface/EffortJointInterface</hardwareInterface>
+      <mechanicalReduction>50</mechanicalReduction>
+    </actuator>
+  </transmission>
+  <!-- #################### -->
+  <transmission name="tran_right_front_wheel">
+    <type>transmission_interface/SimpleTransmission</type>
+    <joint name="joint_right_front_wheel">
+      <hardwareInterface>hardware_interface/EffortJointInterface</hardwareInterface>
+    </joint>
+    <actuator name="motor_right_front_wheel">
+      <hardwareInterface>hardware_interface/EffortJointInterface</hardwareInterface>
+      <mechanicalReduction>50</mechanicalReduction>
+    </actuator>
+  </transmission>
+  <!-- #################### -->
+  <transmission name="tran_right_back_wheel">
+    <type>transmission_interface/SimpleTransmission</type>
+    <joint name="joint_right_back_wheel">
+      <hardwareInterface>hardware_interface/EffortJointInterface</hardwareInterface>
+    </joint>
+    <actuator name="motor_right_back_wheel">
+      <hardwareInterface>hardware_interface/EffortJointInterface</hardwareInterface>
+      <mechanicalReduction>50</mechanicalReduction>
+    </actuator>
+  </transmission>
+  <!-- #################### -->
+  <transmission name="tran_left_front_wheel">
+    <type>transmission_interface/SimpleTransmission</type>
+    <joint name="joint_left_front_wheel">
+      <hardwareInterface>hardware_interface/EffortJointInterface</hardwareInterface>
+    </joint>
+    <actuator name="motor_left_front_wheel">
+      <hardwareInterface>hardware_interface/EffortJointInterface</hardwareInterface>
+      <mechanicalReduction>50</mechanicalReduction>
+    </actuator>
+  </transmission>
+  <!-- #################### -->
+  <transmission name="tran_left_back_wheel">
+    <type>transmission_interface/SimpleTransmission</type>
+    <joint name="joint_left_back_wheel">
+      <hardwareInterface>hardware_interface/EffortJointInterface</hardwareInterface>
+    </joint>
+    <actuator name="motor_left_back_wheel">
       <hardwareInterface>hardware_interface/EffortJointInterface</hardwareInterface>
       <mechanicalReduction>50</mechanicalReduction>

Commit message: add moving control by using keyboard

File: car_model/robots/car_model.xacro (robot description, xacro)
@@ -2,9 +2,9 @@
 <robot name="car_model" xmlns:xacro="http://www.ros.org/wiki/xacro">
   <xacro:property name="PI" value="3.1415926"/>
-  <xacro:property name="car_mass" value="100.0" />
+  <xacro:property name="car_mass" value="1.0" />
   <xacro:property name="car_a" value="0.25" />
   <xacro:property name="car_b" value="0.16" />
   <xacro:property name="car_c" value="0.05" />
-  <xacro:property name="wheel_mass" value="10.0" />
+  <xacro:property name="wheel_mass" value="0.1" />
   <xacro:property name="wheel_lenth" value="0.02" />
   <xacro:property name="wheel_radius" value="0.025" />
@@ -13,5 +13,5 @@
   <xacro:property name="column_height2" value="0.1" />
   <xacro:property name="column_height3" value="0.05" />
-  <xacro:property name="column_mass" value="10.0" />
+  <xacro:property name="column_mass" value="0.1" />
   <xacro:property name="camera_width" value="0.025" />
   <!-- #################### -->
@@ -65,6 +65,17 @@
         rpy="0 0 0" />
       <geometry>
-        <cylinder length="${wheel_lenth}" radius="${wheel_radius}" />
-      </geometry>
+        <!--<cylinder length="${wheel_lenth}" radius="${wheel_radius}" />-->
+        <box size="${wheel_radius*2} ${wheel_radius*2} ${wheel_lenth}" />
+      </geometry>
+      <surface>
+        <friction>
+          <ode>
+            <mu>0</mu>
+            <mu2>0</mu2>
+            <slip1>1.0</slip1>
+            <slip2>1.0</slip2>
+          </ode>
+        </friction>
+      </surface>
     </collision>
     <inertial>
@@ -83,5 +94,6 @@
     <visual>
       <geometry>
-        <cylinder length="${wheel_lenth}" radius="${wheel_radius}" />
+        <!--<cylinder length="${wheel_lenth}" radius="${wheel_radius}" />-->
+        <box size="${wheel_radius*2} ${wheel_radius*2} ${wheel_lenth}" />
       </geometry>
       <material name="grey">
@@ -95,7 +107,7 @@
     <parent link="car_body" />
     <child link="right_front_wheel" />
-    <origin rpy="0 1.57075 1.57075" xyz="${car_a/2-0.02} ${-car_b/2-0.01} 0" />
+    <origin rpy="0 ${PI/2} ${PI/2}" xyz="${car_a/2-0.02} ${-car_b/2-0.01} 0" />
     <limit effort="100" velocity="100" />
-    <joint_properties damping="0" friction="0.0" />
+    <joint_properties damping="0" friction="100" />
   </joint>
   <!-- #################### -->
@@ -106,6 +118,17 @@
         rpy="0 0 0" />
       <geometry>
-        <cylinder length="${wheel_lenth}" radius="${wheel_radius}" />
-      </geometry>
+        <!--<cylinder length="${wheel_lenth}" radius="${wheel_radius}" />-->
+        <box size="${wheel_radius*2} ${wheel_radius*2} ${wheel_lenth}" />
+      </geometry>
+      <surface>
+        <friction>
+          <ode>
+            <mu>0</mu>
+            <mu2>0</mu2>
+            <slip1>1.0</slip1>
+            <slip2>1.0</slip2>
+          </ode>
+        </friction>
+      </surface>
     </collision>
     <inertial>
@@ -124,5 +147,6 @@
     <visual>
       <geometry>
-        <cylinder length="${wheel_lenth}" radius="${wheel_radius}" />
+        <!--<cylinder length="${wheel_lenth}" radius="${wheel_radius}" />-->
+        <box size="${wheel_radius*2} ${wheel_radius*2} ${wheel_lenth}" />
       </geometry>
       <material name="grey">
@@ -136,7 +160,7 @@
     <parent link="car_body" />
     <child link="right_back_wheel" />
-    <origin rpy="0 1.57075 1.57075" xyz="${-car_a/2+0.02} ${-car_b/2-0.01} 0" />
+    <origin rpy="0 ${PI/2} ${PI/2}" xyz="${-car_a/2+0.02} ${-car_b/2-0.01} 0" />
     <limit effort="100" velocity="100" />
-    <joint_properties damping="0" friction="1.0" />
+    <joint_properties damping="0" friction="100" />
   </joint>
   <!-- #################### -->
@@ -147,6 +171,17 @@
         rpy="0 0 0" />
       <geometry>
-        <cylinder length="${wheel_lenth}" radius="${wheel_radius}" />
-      </geometry>
+        <!--<cylinder length="${wheel_lenth}" radius="${wheel_radius}" />-->
+        <box size="${wheel_radius*2} ${wheel_radius*2} ${wheel_lenth}" />
+      </geometry>
+      <surface>
+        <friction>
+          <ode>
+            <mu>0</mu>
+            <mu2>0</mu2>
+            <slip1>1.0</slip1>
+            <slip2>1.0</slip2>
+          </ode>
+        </friction>
+      </surface>
     </collision>
     <inertial>
@@ -165,5 +200,6 @@
     <visual>
       <geometry>
-        <cylinder length="${wheel_lenth}" radius="${wheel_radius}" />
+        <!--<cylinder length="${wheel_lenth}" radius="${wheel_radius}" />-->
+        <box size="${wheel_radius*2} ${wheel_radius*2} ${wheel_lenth}" />
       </geometry>
       <material name="grey">
@@ -177,7 +213,7 @@
     <parent link="car_body" />
     <child link="left_front_wheel" />
-    <origin rpy="0 1.57075 1.57075" xyz="${car_a/2-0.02} ${car_b/2+0.01} 0" />
+    <origin rpy="0 ${PI/2} ${PI/2}" xyz="${car_a/2-0.02} ${car_b/2+0.01} 0" />
     <limit effort="100" velocity="100" />
-    <joint_properties damping="0" friction="1.0" />
+    <joint_properties damping="0" friction="100" />
   </joint>
   <!-- #################### -->
@@ -188,6 +224,17 @@
         rpy="0 0 0" />
       <geometry>
-        <cylinder length="${wheel_lenth}" radius="${wheel_radius}" />
-      </geometry>
+        <!--<cylinder length="${wheel_lenth}" radius="${wheel_radius}" />-->
+        <box size="${wheel_lenth} ${wheel_radius} ${wheel_radius}" />
+      </geometry>
+      <surface>
+        <friction>
+          <ode>
+            <mu>0</mu>
+            <mu2>0</mu2>
+            <slip1>1.0</slip1>
+            <slip2>1.0</slip2>
+          </ode>
+        </friction>
+      </surface>
     </collision>
     <inertial>
@@ -206,5 +253,6 @@
     <visual>
       <geometry>
-        <cylinder length="${wheel_lenth}" radius="${wheel_radius}" />
+        <!--<cylinder length="${wheel_lenth}" radius="${wheel_radius}" />-->
+        <box size="${wheel_radius*2} ${wheel_radius*2} ${wheel_lenth}" />
       </geometry>
       <material name="grey">
@@ -218,7 +266,7 @@
     <parent link="car_body" />
     <child link="left_back_wheel" />
-    <origin rpy="0 1.57075 1.57075" xyz="${-car_a/2+0.02} ${car_b/2+0.01} 0" />
+    <origin rpy="0 ${PI/2} ${PI/2}" xyz="${-car_a/2+0.02} ${car_b/2+0.01} 0" />
     <limit effort="100" velocity="100" />
-    <joint_properties damping="0" friction="1.0" />
+    <joint_properties damping="0" friction="100" />
   </joint>
   <!-- #################### -->
@@ -263,5 +311,5 @@
     <origin xyz="${car_a/2-column_width} 0 ${car_c}" />
     <limit effort="100" velocity="100" />
-    <joint_properties damping="0" friction="1.0" />
+    <joint_properties damping="0" friction="0" />
   </joint>
   <!-- #################### -->
@@ -307,5 +355,5 @@
     <origin xyz="0 0 ${column_height1 - column_width}" />
     <limit effort="100" velocity="100" />
-    <joint_properties damping="0" friction="0.0" />
+    <joint_properties damping="0" friction="0" />
   </joint>
   <!-- #################### -->
@@ -350,5 +398,5 @@
     <origin xyz="0 0 ${column_height2 - column_width}" />
     <limit effort="100" velocity="100" />
-    <joint_properties damping="0" friction="0.0" />
+    <joint_properties damping="0" friction="0" />
   </joint>
   <!-- #################### -->
@@ -382,4 +430,8 @@
   </joint>
   <!-- #################### -->
+  <gazebo reference="world_link">
+    <material>Gazebo/Yellow</material>
+    <!--<turnGravityOff>false<turnGravityOff>-->
+  </gazebo>
   <gazebo reference="car_body">
     <material>Gazebo/Orange</material>
@@ -433,5 +485,5 @@
     <actuator name="motor_column_link1">
       <hardwareInterface>hardware_interface/EffortJointInterface</hardwareInterface>
-      <mechanicalReduction>50</mechanicalReduction>
+      <mechanicalReduction>1</mechanicalReduction>
     </actuator>
   </transmission>
@@ -444,5 +496,5 @@
     <actuator name="motor_column_link2">
       <hardwareInterface>hardware_interface/EffortJointInterface</hardwareInterface>
-      <mechanicalReduction>50</mechanicalReduction>
+      <mechanicalReduction>1</mechanicalReduction>
     </actuator>
   </transmission>
@@ -455,5 +507,5 @@
     <actuator name="motor_column_link3">
       <hardwareInterface>hardware_interface/EffortJointInterface</hardwareInterface>
-      <mechanicalReduction>50</mechanicalReduction>
+      <mechanicalReduction>1</mechanicalReduction>
     </actuator>
   </transmission>
@@ -466,5 +518,5 @@
     <actuator name="motor_right_front_wheel">
       <hardwareInterface>hardware_interface/EffortJointInterface</hardwareInterface>
-      <mechanicalReduction>50</mechanicalReduction>
+      <mechanicalReduction>1</mechanicalReduction>
     </actuator>
   </transmission>
@@ -477,5 +529,5 @@
     <actuator name="motor_right_back_wheel">
       <hardwareInterface>hardware_interface/EffortJointInterface</hardwareInterface>
-      <mechanicalReduction>50</mechanicalReduction>
+      <mechanicalReduction>1</mechanicalReduction>
     </actuator>
   </transmission>
@@ -488,5 +540,5 @@
     <actuator name="motor_left_front_wheel">
       <hardwareInterface>hardware_interface/EffortJointInterface</hardwareInterface>
-      <mechanicalReduction>50</mechanicalReduction>
+      <mechanicalReduction>1</mechanicalReduction>
     </actuator>
   </transmission>
@@ -499,5 +551,5 @@
     <actuator name="motor_left_back_wheel">
       <hardwareInterface>hardware_interface/EffortJointInterface</hardwareInterface>
-      <mechanicalReduction>50</mechanicalReduction>
+      <mechanicalReduction>1</mechanicalReduction>
     </actuator>
   </transmission>
@@ -523,5 +575,6 @@
         </noise>
       </camera>
-      <plugin name="camera_controller" filename="libgazebo_ros_camera.so">
+      <plugin name="camera_controller"
+        filename="libgazebo_ros_camera.so">
         <alwaysOn>true</alwaysOn>
         <updateRate>0.0</updateRate>
@@ -545,5 +598,31 @@
   <!-- #################### -->
   <gazebo>
-    <plugin name="gazebo_ros_control" filename="libgazebo_ros_control.so">
+    <plugin name="skid_steer_drive_controller"
+      filename="libgazebo_ros_skid_steer_drive.so">
+      <alwaysOn>true</alwaysOn>
+      <updateRate>100.0</updateRate>
+      <robotNamespace>/</robotNamespace>
+      <rightFrontJoint>joint_right_front_wheel</rightFrontJoint>
+      <rightRearJoint>joint_right_back_wheel</rightRearJoint>
+      <leftFrontJoint>joint_left_front_wheel</leftFrontJoint>
+      <leftRearJoint>joint_left_back_wheel</leftRearJoint>
+      <wheelSeparation>${car_b}</wheelSeparation>
+      <wheelDiameter>${wheel_radius*2}</wheelDiameter>
+      <commandTopic>cmd_vel</commandTopic>
+      <odometryTopic>odom</odometryTopic>
+      <robotBaseFrame>world_link</robotBaseFrame>
+      <odometryFrame>odom</odometryFrame>
+      <covariance_x>0.000100</covariance_x>
+      <covariance_y>0.000100</covariance_y>
+      <covariance_yaw>0.010000</covariance_yaw>
+      <torque>1</torque>
+      <topicName>cmd_vel</topicName>
+      <broadcastTF>1</broadcastTF>
+    </plugin>
+  </gazebo>
+  <!-- #################### -->
+  <gazebo>
+    <plugin name="gazebo_ros_control"
+      filename="libgazebo_ros_control.so">
       <robotNamespace>/car_model</robotNamespace>
       <robotSimType>gazebo_ros_control/DefaultRobotHWSim</robotSimType>

Commit message: add map

File: car_model/robots/car_model.xacro (robot description, xacro)
@@ -65,6 +65,6 @@
         rpy="0 0 0" />
       <geometry>
-        <!--<cylinder length="${wheel_lenth}" radius="${wheel_radius}" />-->
-        <box size="${wheel_radius*2} ${wheel_radius*2} ${wheel_lenth}" />
+        <cylinder length="${wheel_lenth}" radius="${wheel_radius}" />
+        <!--<box size="${wheel_radius*2} ${wheel_radius*2} ${wheel_lenth}" />-->
       </geometry>
       <surface>
@@ -109,5 +109,5 @@
     <origin rpy="0 ${PI/2} ${PI/2}" xyz="${car_a/2-0.02} ${-car_b/2-0.01} 0" />
     <limit effort="100" velocity="100" />
-    <joint_properties damping="0" friction="100" />
+    <joint_properties damping="0" friction="0" />
   </joint>
   <!-- #################### -->
@@ -118,6 +118,6 @@
         rpy="0 0 0" />
       <geometry>
-        <!--<cylinder length="${wheel_lenth}" radius="${wheel_radius}" />-->
-        <box size="${wheel_radius*2} ${wheel_radius*2} ${wheel_lenth}" />
+        <cylinder length="${wheel_lenth}" radius="${wheel_radius}" />
+        <!--<box size="${wheel_radius*2} ${wheel_radius*2} ${wheel_lenth}" />-->
       </geometry>
       <surface>
@@ -162,5 +162,5 @@
     <origin rpy="0 ${PI/2} ${PI/2}" xyz="${-car_a/2+0.02} ${-car_b/2-0.01} 0" />
     <limit effort="100" velocity="100" />
-    <joint_properties damping="0" friction="100" />
+    <joint_properties damping="0" friction="0" />
   </joint>
   <!-- #################### -->
@@ -171,6 +171,6 @@
         rpy="0 0 0" />
       <geometry>
-        <!--<cylinder length="${wheel_lenth}" radius="${wheel_radius}" />-->
-        <box size="${wheel_radius*2} ${wheel_radius*2} ${wheel_lenth}" />
+        <cylinder length="${wheel_lenth}" radius="${wheel_radius}" />
+        <!--<box size="${wheel_radius*2} ${wheel_radius*2} ${wheel_lenth}" />-->
       </geometry>
       <surface>
@@ -215,5 +215,5 @@
     <origin rpy="0 ${PI/2} ${PI/2}" xyz="${car_a/2-0.02} ${car_b/2+0.01} 0" />
     <limit effort="100" velocity="100" />
-    <joint_properties damping="0" friction="100" />
+    <joint_properties damping="0" friction="0" />
   </joint>
   <!-- #################### -->
@@ -224,6 +224,6 @@
         rpy="0 0 0" />
       <geometry>
-        <!--<cylinder length="${wheel_lenth}" radius="${wheel_radius}" />-->
-        <box size="${wheel_lenth} ${wheel_radius} ${wheel_radius}" />
+        <cylinder length="${wheel_lenth}" radius="${wheel_radius}" />
+        <!--<box size="${wheel_radius*2} ${wheel_radius*2} ${wheel_lenth}" />-->
       </geometry>
       <surface>
@@ -268,5 +268,5 @@
     <origin rpy="0 ${PI/2} ${PI/2}" xyz="${-car_a/2+0.02} ${car_b/2+0.01} 0" />
     <limit effort="100" velocity="100" />
-    <joint_properties damping="0" friction="100" />
+    <joint_properties damping="0" friction="0" />
   </joint>
   <!-- #################### -->

Commit message: add column controling by keyboard and move car_control into car_model

File: car_model/robots/car_model.xacro (robot description, xacro)
@@ -10,6 +10,6 @@
   <xacro:property name="wheel_radius" value="0.025" />
   <xacro:property name="column_width" value="0.02" />
-  <xacro:property name="column_height1" value="0.2" />
-  <xacro:property name="column_height2" value="0.1" />
+  <xacro:property name="column_height1" value="0.05" />
+  <xacro:property name="column_height2" value="0.2" />
   <xacro:property name="column_height3" value="0.05" />
   <xacro:property name="column_mass" value="0.1" />
@@ -305,6 +305,7 @@
     </inertial>
   </link>
+  <!-- #################### -->
   <joint name="joint_column_link1" type="continuous">
-    <axis xyz="0 1 0" rpy="0 0 0" />
+    <axis xyz="0 0 1" rpy="0 0 0" />
     <parent link="car_body" />
     <child link="column_link1" />
@@ -392,4 +393,5 @@
     </inertial>
   </link>
+  <!-- #################### -->
   <joint name="joint_column_link3" type="continuous">
     <axis xyz="0 0 1" rpy="0 0 0" />
@@ -425,5 +427,5 @@
   <!-- #################### -->
   <joint name="joint_camera_link" type="fixed">
-    <origin xyz="0 0 ${column_height3}" rpy="${-PI/2} 0 ${-PI/2}"/>
+    <origin xyz="0 0 ${column_height3}" rpy="0 ${-PI/2} 0"/>
     <parent link="column_link3"/>
     <child link="camera_link"/>
@@ -486,4 +488,5 @@
       <hardwareInterface>hardware_interface/EffortJointInterface</hardwareInterface>
       <mechanicalReduction>1</mechanicalReduction>
+      <motorTorqueConstant>1</motorTorqueConstant>
     </actuator>
   </transmission>
@@ -497,4 +500,5 @@
       <hardwareInterface>hardware_interface/EffortJointInterface</hardwareInterface>
       <mechanicalReduction>1</mechanicalReduction>
+      <motorTorqueConstant>1</motorTorqueConstant>
     </actuator>
   </transmission>
@@ -508,4 +512,5 @@
       <hardwareInterface>hardware_interface/EffortJointInterface</hardwareInterface>
       <mechanicalReduction>1</mechanicalReduction>
+      <motorTorqueConstant>1</motorTorqueConstant>
     </actuator>
   </transmission>
